File: hw_2/Blue_Pill_Clone.sch (KiCad schematic (older format))
At the start: 43 parts, among them J2 Conn_01x04_Male, J3 USB_B_Micro, J8 Conn_01x04_Male, SW1 SW_Push, U1 MIC5504-3.3YM5, U2 STM32F103C8Tx, Y2 8MHz, Y3 32.768k

Commit message: Version 1.0 as ordered
Parts:
- Y3: LCSC C32346 -> C48615
Changed lines of the file:
@@
 F 2 "Crystal:Crystal_SMD_3215-2Pin_3.2x1.5mm" H 5900 6900 50  0001 C CNN
 F 3 "~" H 5900 6900 50  0001 C CNN
-F 4 "C32346" V 5900 6900 50  0001 C CNN "LCSC"
+F 4 "C48615" V 5900 6900 50  0001 C CNN "LCSC"
 	1    5900 6900
 	0    1    1    0
